File: UDOO-Connectivity-Shield/XBEE_NFC_shield_v0_2.brd (EAGLE design)
At the start: 99.1 x 53.3 mm, 15 parts, among them U1 XBEE

Commit message: Add Info on the shield
Other:
- board size 99.1 x 53.3 mm -> 102.6 x 53.3 mm
- board text added: "ADAFRUIT_NFC_SHIELD"
- board text added: "CONNECTIVITY"
- board text added: "Francesco Ermini"
- board text added: "SCHIELD"
- board text added: "SPI HEADER"
- board text added: "UDOO"
- board text added: "by"
Changed lines of the file:
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@@
 <text x="58.166" y="39.878" size="1.778" layer="37" rot="R90">GND</text>
 <text x="6.731" y="6.477" size="1.778" layer="37">SS</text>
+<text x="73.787" y="50.165" size="1.778" layer="37">SPI HEADER </text>
+<text x="-1.143" y="16.002" size="1.778" layer="37" rot="R90">ADAFRUIT_NFC_SHIELD</text>
+<wire x1="26.67" y1="4.572" x2="26.797" y2="4.445" width="0.4064" layer="20"/>
+<wire x1="26.797" y1="4.445" x2="94.742" y2="4.445" width="0.4064" layer="20"/>
+<wire x1="94.742" y1="4.445" x2="94.869" y2="4.572" width="0.4064" layer="20"/>
+<wire x1="94.869" y1="4.572" x2="94.869" y2="49.149" width="0.4064" layer="20"/>
+<wire x1="94.869" y1="49.149" x2="94.488" y2="49.53" width="0.4064" layer="20"/>
+<wire x1="94.488" y1="49.53" x2="0.254" y2="49.53" width="0.4064" layer="20"/>
+<wire x1="0.254" y1="49.53" x2="-3.556" y2="45.72" width="0.4064" layer="20"/>
+<wire x1="-3.556" y1="45.72" x2="-3.556" y2="4.572" width="0.4064" layer="20"/>
+<wire x1="-3.556" y1="4.572" x2="-3.302" y2="4.318" width="0.4064" layer="20"/>
+<wire x1="-3.302" y1="4.318" x2="44.323" y2="4.318" width="0.4064" layer="20"/>
+<text x="81.026" y="24.638" size="1.778" layer="20">UDOO</text>
+<text x="70.358" y="19.685" size="1.778" layer="20">CONNECTIVITY</text>
+<text x="77.597" y="16.256" size="1.778" layer="20">SCHIELD</text>
+<text x="70.485" y="9.652" size="1.778" layer="20">Francesco Ermini</text>
+<text x="81.534" y="13.208" size="1.778" layer="20">by</text>
 </plain>
 <attributes>
